File: i.MX8X Flight Computer Carrier Board/CADENCE i.MX8X Carrier Board rev1/Control.kicad_sch (KiCad schematic)
At the start: 20 parts, among them SW1 SW_DIP_x01, SW2 KMR221GLFS, SW3 SW_DIP_x04

Commit message: Added in the DIP switches for the BOM, did some DRC
Parts:
- SW3: footprint Footprints:SW_1571983-4 -> Footprints:SW-SMD_8P-L11.3-W6.2-P1.27-LS8.2
Changed lines of the file:
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@@
 			)
 		)
-		(property "Footprint" "Footprints:SW_1571983-4"
+		(property "Footprint" "Footprints:SW-SMD_8P-L11.3-W6.2-P1.27-LS8.2"
 			(at 142.24 45.72 0)
 			(effects
@@
 			)
 		)
-		(property "Description" "4x DIP Switch, Single Pole Single Throw (SPST) switch, small symbol"
+		(property "Description" "https://www.lcsc.com/product-detail/C266192.html?s_z=n_q_x_%2509%25201571983-4&spm=wm.ssy.em.0.tz&lcsc_vid=QgdeBFICFlVZAlBfRFdaXgZXQwdeUlMAQFgIBVJTQwUxVlNeQ1JbVldeR1RaXjsOAxUeFF5JWBYZEEoKFBINSQcJGk4dAgUUFAk%3D"
 			(at 142.24 45.72 0)
 			(effects
