File: i.MX8X Flight Computer Carrier Board/CADENCE i.MX8X Carrier Board rev1/uSD.kicad_sch (KiCad schematic)
At the start: 18 parts, among them U8 BD2204GUL-E2

Commit message: replaced obsolete uSD
need to recreate fab files
Parts:
- Card1: value 5027740891 -> HRS DM3BT-DSF-PEJS; footprint imx8_carrier_board_footprints:TF-SMD_5027740891 -> uSD:HRS_DM3BT-DSF-PEJS; LCSC Part C330255 -> C597972
