File: i.MX8X Flight Computer Carrier Board/CADENCE i.MX8X Carrier Board rev1/Peripherals.kicad_sch (KiCad schematic)
At the start: 14 parts, among them U23 RV-3028-C7, U24 LSM6DSO, U25 LIS2MDL, U26 TMP112xxDRL, U27 INA219AxDCN

Commit message: Replaced with IIS2MDCTR
Parts:
- U25: value LIS2MDL -> IIS2MDCTR
Changed lines of the file:
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@@
 			)
 		)
-		(property "Value" "LIS2MDL"
+		(property "Value" "IIS2MDCTR"
 			(at 134.874 89.154 0)
 			(show_name no)
