File: i.MX8X Flight Computer Carrier Board/CADENCE i.MX8X Carrier Board rev1/CADENCE i.MX8X Carrier Board rev1.kicad_pcb (KiCad board)
At the start: 6 copper layers, 172 x 85 mm, 431 parts, among them CN1 DF11-16DP-2DSA(08), CN2 DF11-16DP-2DSA(08), CN3 DF11-16DP-2DSA(08), CN4 DF11-16DP-2DSA(08), J1 BTH-070-02-L-D-A, J10 Conn_01x04, J11 Conn_01x04, J16 Conn_01x04, J17 Conn_01x04, J2 USB_C_Receptacle_USB2.0_16P, J21 Conn_02x02_Odd_Even, J22 Conn_01x04, J3 USB_A, J4 Conn_Coaxial, J5 USB_C_Receptacle_USB2.0_16P, J6 Conn_01x01, J7 Conn_01x08, J8 Conn_02x26_Odd_Even, J9 Conn_02x26_Odd_Even, Q1 IRLML6401, Q2 BSS138, Q3 BSS138, SW1 SW_DIP_x01, SW2 KMR221GLFS, SW3 SW_DIP_x04, SW4 SW_DIP_x01, T1 WE-RJ45_7499111121A, T2 WE-RJ45_7499111121A, U1 LT8612, U10 ZDSD04GLGEAG, U11 MR20H40, U12 MR20H40, U13 DP83867IRRGZR, U14 74LVC2G07, U15 USBLC6-2SC6, U16 USBLC6-2SC6, U17 SN65C1168ERGYR, U18 P82B715DR, U19 P82B715DR, U2 LT8612, U20 P82B715DR, U21 INA219AxDCN, U22 Skytraq Orion B16 GPS, U23 RV-3028-C7, U24 LSM6DSO, U25 IIS2MDCTR, U26 TMP112xxDRL, U27 INA219AxDCN, U28 LP38693MP-ADJ/NOPB, U29 74CBTLV3257BQ, U3 TPS22975, U30 CAT93C66VI-GT3, U31 USBLC6-2SC6, U32 FT2232HL, U33 SN65HVD233, U34 INA219AxDCN, U35 TPS22810DBV, U36 INA219AxDCN, U37 TPS22810DBV, U38 INA219AxDCN, U39 TPS22975, U4 LT3115-1, U40 TXS0101DCKR, U41 TXS0101DCKR, U5 TLV71325PDQNR, U6 TLV71310PDQNR, U7 TLV1704, U8 BD2204GUL-E2, U9 MX25UM51245G, Y1 25MHz, Y2 12MHz

Commit message: Replaced 0402W with C159987
Parts:
- Card1: value 5027740891 -> HRS DM3BT-DSF-PEJS
Changed lines of the file:
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@@
 			)
 		)
-		(attr exclude_from_pos_files exclude_from_bom)
 		(duplicate_pad_numbers_are_jumpers no)
 		(fp_line
@@
 			)
 		)
-		(attr exclude_from_pos_files exclude_from_bom)
 		(duplicate_pad_numbers_are_jumpers no)
 		(fp_line
@@
 			)
 		)
-		(attr exclude_from_pos_files exclude_from_bom)
 		(duplicate_pad_numbers_are_jumpers no)
 		(fp_line
@@
 			)
 		)
-		(attr exclude_from_pos_files exclude_from_bom)
 		(duplicate_pad_numbers_are_jumpers no)
 		(fp_line
@@
 			)
 		)
-		(attr exclude_from_pos_files exclude_from_bom)
 		(duplicate_pad_numbers_are_jumpers no)
 		(fp_line
@@
 			)
 		)
-		(attr exclude_from_pos_files exclude_from_bom)
 		(duplicate_pad_numbers_are_jumpers no)
 		(fp_line
@@
 			)
 		)
-		(attr exclude_from_pos_files exclude_from_bom)
 		(duplicate_pad_numbers_are_jumpers no)
 		(fp_line
@@
 		)
 		(clearance 0.2)
-		(attr through_hole exclude_from_pos_files exclude_from_bom)
+		(attr through_hole)
 		(duplicate_pad_numbers_are_jumpers no)
 		(fp_line
@@
 			)
 		)
-		(attr exclude_from_pos_files exclude_from_bom)
 		(duplicate_pad_numbers_are_jumpers no)
 		(fp_line
@@
 			)
 		)
-		(attr through_hole exclude_from_pos_files exclude_from_bom)
+		(attr through_hole)
 		(duplicate_pad_numbers_are_jumpers no)
 		(fp_line
@@
 		)
 		(clearance 0.2)
-		(attr through_hole exclude_from_pos_files exclude_from_bom)
+		(attr through_hole)
 		(duplicate_pad_numbers_are_jumpers no)
 		(fp_line
@@
 			)
 		)
-		(attr exclude_from_pos_files exclude_from_bom)
 		(duplicate_pad_numbers_are_jumpers no)
 		(fp_line
@@
 			)
 		)
-		(attr smd exclude_from_pos_files exclude_from_bom)
+		(attr smd)
 		(duplicate_pad_numbers_are_jumpers no)
 		(fp_circle
@@
 			)
 		)
-		(attr exclude_from_pos_files exclude_from_bom)
 		(duplicate_pad_numbers_are_jumpers no)
 		(fp_line
@@
 			)
 		)
-		(attr exclude_from_pos_files exclude_from_bom)
 		(duplicate_pad_numbers_are_jumpers no)
 		(fp_line
@@
 		)
 		(zone_connect 1)
-		(attr exclude_from_pos_files exclude_from_bom allow_soldermask_bridges)
+		(attr allow_soldermask_bridges)
 		(duplicate_pad_numbers_are_jumpers no)
 		(fp_rect
@@
 			)
 		)
-		(attr exclude_from_pos_files exclude_from_bom)
 		(duplicate_pad_numbers_are_jumpers no)
 		(fp_line
@@
 			)
 		)
-		(property "LCSC" "C474132"
+		(property "LCSC" "C159987"
 			(at 0 0 0)
 			(unlocked yes)
@@
 			)
 		)
-		(attr through_hole exclude_from_pos_files exclude_from_bom)
+		(attr through_hole)
 		(duplicate_pad_numbers_are_jumpers no)
 		(fp_line
@@
 			)
 		)
-		(attr smd exclude_from_pos_files exclude_from_bom)
+		(attr smd)
 		(duplicate_pad_numbers_are_jumpers no)
 		(fp_circle
@@
 			)
 		)
-		(attr exclude_from_pos_files exclude_from_bom)
 		(duplicate_pad_numbers_are_jumpers no)
 		(fp_line
@@
 			)
 		)
-		(attr smd exclude_from_pos_files exclude_from_bom)
+		(attr smd)
 		(duplicate_pad_numbers_are_jumpers no)
 		(fp_line
@@
 			)
 		)
-		(attr through_hole exclude_from_pos_files exclude_from_bom)
+		(attr through_hole)
 		(duplicate_pad_numbers_are_jumpers no)
 		(fp_line
@@
 			)
 		)
-		(attr exclude_from_pos_files exclude_from_bom)
 		(duplicate_pad_numbers_are_jumpers no)
 		(fp_line
@@
 			)
 		)
-		(attr exclude_from_pos_files exclude_from_bom)
 		(duplicate_pad_numbers_are_jumpers no)
 		(fp_line
@@
 			)
 		)
-		(attr exclude_from_pos_files exclude_from_bom)
 		(duplicate_pad_numbers_are_jumpers no)
 		(fp_line
@@
 			)
 		)
-		(attr through_hole exclude_from_pos_files exclude_from_bom)
+		(attr through_hole)
 		(duplicate_pad_numbers_are_jumpers no)
 		(fp_line
@@
 			)
 		)
-		(attr through_hole exclude_from_pos_files exclude_from_bom)
+		(attr through_hole)
 		(duplicate_pad_numbers_are_jumpers no)
 		(fp_line
@@
 		)
 		(zone_connect 1)
-		(attr exclude_from_pos_files exclude_from_bom allow_soldermask_bridges)
+		(attr allow_soldermask_bridges)
 		(duplicate_pad_numbers_are_jumpers no)
 		(fp_rect
@@
 		)
 		(zone_connect 1)
-		(attr exclude_from_pos_files exclude_from_bom allow_soldermask_bridges)
+		(attr allow_soldermask_bridges)
 		(duplicate_pad_numbers_are_jumpers no)
 		(fp_rect
@@
 			)
 		)
-		(attr exclude_from_pos_files exclude_from_bom)
 		(duplicate_pad_numbers_are_jumpers no)
 		(fp_line
@@
 			)
 		)
-		(attr through_hole exclude_from_pos_files exclude_from_bom)
+		(attr through_hole)
 		(duplicate_pad_numbers_are_jumpers no)
 		(fp_line
@@
 			)
 		)
-		(attr exclude_from_pos_files exclude_from_bom)
 		(duplicate_pad_numbers_are_jumpers no)
 		(fp_line
@@
 			)
 		)
-		(attr exclude_from_pos_files exclude_from_bom)
 		(duplicate_pad_numbers_are_jumpers no)
 		(fp_line
@@
 			)
 		)
-		(attr exclude_from_pos_files exclude_from_bom)
 		(duplicate_pad_numbers_are_jumpers no)
 		(fp_line
@@
 			)
 		)
-		(attr exclude_from_pos_files exclude_from_bom)
 		(duplicate_pad_numbers_are_jumpers no)
 		(fp_line
@@
 			)
 		)
-		(attr exclude_from_pos_files exclude_from_bom)
 		(duplicate_pad_numbers_are_jumpers no)
 		(fp_line
@@
 			)
 		)
-		(attr exclude_from_pos_files exclude_from_bom)
 		(duplicate_pad_numbers_are_jumpers no)
 		(fp_line
@@
 			)
 		)
-		(attr exclude_from_pos_files exclude_from_bom)
 		(duplicate_pad_numbers_are_jumpers no)
 		(fp_line
@@
 			)
 		)
-		(property "Value" "5027740891"
+		(property "Value" "HRS DM3BT-DSF-PEJS"
 			(at 4.8446 -17.1296 0)
 			(layer "B.Fab")
@@
 			)
 		)
-		(attr smd exclude_from_pos_files exclude_from_bom)
+		(attr smd)
 		(duplicate_pad_numbers_are_jumpers no)
 		(fp_poly
