File: i.MX8X Flight Computer Carrier Board/CADENCE i.MX8X Carrier Board rev1/Watchdog.kicad_sch (KiCad schematic)
At the start: 36 parts, among them U7 TLV1704

Commit message: Replaced 0402W with C159987
Parts:
- R39: LCSC C474132 -> C159987
Changed lines of the file:
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@@
 			)
 		)
-		(property "LCSC" "C474132"
+		(property "LCSC" "C159987"
 			(at 186.182 124.46 0)
 			(hide yes)
