File: i.MX8X Flight Computer Carrier Board/CADENCE i.MX8X Carrier Board rev1/CADENCE i.MX8X Carrier Board rev1.kicad_sch (KiCad schematic)
At the start: 0 parts

Commit message: schematic cleanup & 3d model updates
put in more 3d models & cleaned up schematic organization.

3d model assignment breaks with KiCAD library footprints/symbols
Other:
- note added: "Bill of Materials and Manufacturing Data generated by Bouni KiCAD plugin: https://github.com/Bouni/kicad-jlcpcb-tools"
- note removed: "PDR Block Diagram ---->>>"
