File: i.MX8X Flight Computer Carrier Board/CADENCE i.MX8X Carrier Board rev1/Power.kicad_sch (KiCad schematic)
At the start: 64 parts, among them U1 LT8612, U2 LT8612, U3 TPS22975, U4 LT3115-1, U5 TLV71325PDQNR, U6 TLV71310PDQNR

Commit message: BOM updates
most ICs and capacitors, some mechanical connectors, etc picked. most remaining components are resistors, connectors (usb, buttons, etc)

max, if you can add the enet connectors u found to the BOm. matthew, if you can add the buttons and USB ports u found to the BOM as well. Matthew, if you can also add the inductors we previously picked earlier last semester too pls.
Other:
- note added: "2x 1210 Ceramic Caps or Tantalum Caps"
- note removed: "2x 1210 Ceramic Caps"
Changed lines of the file:
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@@
 		)
 	)
-	(text "2x 1210 Ceramic Caps"
+	(text "2x 1210 Ceramic Caps or \nTantalum Caps\n"
 		(exclude_from_sim no)
-		(at 139.954 43.942 0)
+		(at 141.732 40.894 0)
 		(effects
 			(font

Commit message: BOM part selection, DRC fixes for traces & shorted vias, fixed power pours mentioned in previous design review
Parts:
- C29, C30, C35: value 0.1uF -> 100nF
Changed lines of the file:
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@@
 			)
 		)
-		(property "Value" "0.1uF"
+		(property "Value" "100nF"
 			(at 273.05 149.352 0)
 			(effects
@@
 			)
 		)
-		(property "Value" "0.1uF"
+		(property "Value" "100nF"
 			(at 212.09 127 0)
 			(effects
@@
 			)
 		)
-		(property "Value" "0.1uF"
+		(property "Value" "100nF"
 			(at 237.744 127 0)
 			(effects
